File: licenta/eagle/Controller/controller_v2.sch (EAGLE design)
At the start: 19 parts, among them IC1 7805T

Commit message: 4 chapters done
Parts:
- added JP2: (no value), pinhead:PINHD-1X2
- added LED1: (no value), led:LED5MM
- added R_LED: 100, rcl:R-EU_0207/10
Connections:
- new net N$12: JP2.1, R_LED.1
- new net N$17: JP2.2, LED1.A
- net GND: now also LED1.C
- net VCC: now also R_LED.2
Changed lines of the file:
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@@
 <part name="GND9" library="supply1" library_urn="urn:adsk.eagle:library:371" deviceset="GND" device=""/>
 <part name="USER_INTERFACE" library="pinhead" library_urn="urn:adsk.eagle:library:325" deviceset="PINHD-1X3" device="" package3d_urn="urn:adsk.eagle:package:22458/2"/>
+<part name="LED1" library="led" library_urn="urn:adsk.eagle:library:259" deviceset="LED" device="5MM" package3d_urn="urn:adsk.eagle:package:15799/2"/>
+<part name="R_LED" library="rcl" library_urn="urn:adsk.eagle:library:334" deviceset="R-EU_" device="0207/10" package3d_urn="urn:adsk.eagle:package:23491/1" value="100"/>
+<part name="P+9" library="supply1" library_urn="urn:adsk.eagle:library:371" deviceset="VCC" device=""/>
+<part name="GND10" library="supply1" library_urn="urn:adsk.eagle:library:371" deviceset="GND" device=""/>
+<part name="JP2" library="pinhead" library_urn="urn:adsk.eagle:library:325" deviceset="PINHD-1X2" device="" package3d_urn="urn:adsk.eagle:package:22435/2"/>
 </parts>
 <sheets>
@@
 <instance part="GND9" gate="1" x="182.88" y="76.2"/>
 <instance part="USER_INTERFACE" gate="A" x="93.98" y="137.16"/>
+<instance part="LED1" gate="G$1" x="43.18" y="147.32"/>
+<instance part="R_LED" gate="G$1" x="43.18" y="167.64" rot="R90"/>
+<instance part="P+9" gate="VCC" x="43.18" y="180.34"/>
+<instance part="GND10" gate="1" x="43.18" y="134.62"/>
+<instance part="JP2" gate="G$1" x="53.34" y="154.94"/>
 </instances>
 <busses>
@@
 <wire x1="182.88" y1="114.3" x2="182.88" y2="119.38" width="0.1524" layer="91"/>
 </segment>
+<segment>
+<pinref part="P+9" gate="VCC" pin="VCC"/>
+<pinref part="R_LED" gate="G$1" pin="2"/>
+<wire x1="43.18" y1="177.8" x2="43.18" y2="172.72" width="0.1524" layer="91"/>
+</segment>
 </net>
 <net name="N$1" class="0">
@@
 <wire x1="182.88" y1="111.76" x2="182.88" y2="78.74" width="0.1524" layer="91"/>
 </segment>
+<segment>
+<pinref part="LED1" gate="G$1" pin="C"/>
+<pinref part="GND10" gate="1" pin="GND"/>
+<wire x1="43.18" y1="142.24" x2="43.18" y2="137.16" width="0.1524" layer="91"/>
+</segment>
 </net>
 <net name="CLK" class="0">
@@
 </segment>
 </net>
+<net name="N$12" class="0">
+<segment>
+<pinref part="R_LED" gate="G$1" pin="1"/>
+<wire x1="43.18" y1="162.56" x2="43.18" y2="157.48" width="0.1524" layer="91"/>
+<pinref part="JP2" gate="G$1" pin="1"/>
+<wire x1="43.18" y1="157.48" x2="50.8" y2="157.48" width="0.1524" layer="91"/>
+</segment>
+</net>
+<net name="N$17" class="0">
+<segment>
+<pinref part="JP2" gate="G$1" pin="2"/>
+<wire x1="50.8" y1="154.94" x2="43.18" y2="154.94" width="0.1524" layer="91"/>
+<pinref part="LED1" gate="G$1" pin="A"/>
+<wire x1="43.18" y1="154.94" x2="43.18" y2="149.86" width="0.1524" layer="91"/>
+</segment>
+</net>
